Commit message: 打通 MTC coke_can 抓取与放置全流程
- moveit_config: planning_plugin → planning_plugins 复数键，request/response
  适配器换 Jazzy 命名；OMPL 切回 IPTP 并给 RRTConnect 设 range=0.5；
  trajectory_execution 放宽到 5×+10s 容忍夹爪闭合反弹；sensors_3d 关
  octomap 防机器人体素污染场景；joint_limits 给 shoulder_lift 加上界 0
  防触地；ros2_controllers 修正 default_tolerance 名称并启用 stall。
- ur.srdf: half_closed 改 0.22 适配 coke_can 直径；补 torso/camera 与
  夹爪 11 个子链接的自碰撞排除。
- ur.ros2_control.xacro / initial_positions: 删除不存在的
  left_outer_knuckle_joint。
- mtc_node: pick 后插入 ModifyPlanningScene 允许被抓物与 arm/torso 碰撞，
  place 前撤销；规划失败时 printState 定位 stage。
- mtc_node_params: max_solutions=5 兼顾稳定性与耗时；cartesian 缩放降
  至 0.3 满足 CLAUDE.md 硬约束；object_dimensions 改成 coke_can 尺寸。
- get_planning_scene_server: crop 收紧排除机器人本体；circle/RANSAC
  阈值放宽，line 检测事实禁用；object_segmentation 在 RANSAC 找不到
  circle 时根据 cluster XY 包围盒长宽比回退生成 circle 参数。
- ur.gazebo.launch.py: GZ_SIM_RESOURCE_PATH 增补 robotiq 与
  ur_description 上层 share，修复夹爪 mesh 缺失。
- world / coke_can: 物理步长 4ms；coke_can 碰撞体改解析圆柱避免 ODE
  trimesh 接触爆炸；world 暂时只保留 coke_can 单一目标。
- intel_rgbd_cam_d435: 相机 5Hz、关闭 GUI 预览渲染。
- vendored MTC: 给 capabilities/core/demo/msgs/rviz_marker_tools/
  visualization 加 COLCON_IGNORE 跳过编译。
- mujoco_ur_rl_ros2: 删除多余的 ament_python buildtool_depend。

Co-Authored-By: Claude Opus 4.7 (1M context) <noreply@anthropic.com>

File: moveit_config/config/ur.ros2_control.xacro (robot description, xacro)
@@ -83,11 +83,6 @@
                  command_interface here fights physics and causes asymmetric finger motion.
                  Per-joint initial_value keys prevent right-side joints from starting at limits. -->
-            <!-- left_outer_knuckle_joint (was missing — added) -->
-            <joint name="left_outer_knuckle_joint">
-                <state_interface name="position">
-                    <param name="initial_value">${initial_positions['left_outer_knuckle_joint']}</param>
-                </state_interface>
-                <state_interface name="velocity"/>
-            </joint>
+            <!-- 注意：本 URDF 的夹爪设计下不存在独立的 left_outer_knuckle_joint，
+                 finger_joint (见上) 就是左外指节主驱动关节。此处保留注释以防误补。 -->
             <!-- right_outer_knuckle_joint -->
             <joint name="right_outer_knuckle_joint">

File: ur_description/urdf/intel_rgbd_cam_d435.urdf.xacro (robot description, xacro)
@@ -144,5 +144,6 @@
     </camera>
     <always_on>1</always_on>
-    <update_rate>10</update_rate>
+    <!-- 相机更新频率 10 Hz → 5 Hz；感知管线只需检测稳定物体，5 Hz 充裕 -->
+    <update_rate>5</update_rate>
     <gz_frame_id>camera_head_link</gz_frame_id>
     <output>
@@ -151,5 +152,6 @@
       <point_cloud>true</point_cloud>
     </output>
-    <visualize>true</visualize>
+    <!-- 关闭 GUI 内的相机预览渲染，省 5–10% RTF；不影响话题数据流 -->
+    <visualize>false</visualize>
   </sensor>
 </gazebo>
